Commit message: fix: Update camera poses according to calib_01 calibration (see pdf in GGDrive/Calibration)

File: jetsonNano/ros2_ws/src/ecosense_description/src/description/ecosense_description.urdf (robot description, URDF)
Before this commit: robot ecosense, 18 links, 17 joints
Joints:
- joint camera_right_joint: origin xyz=${camera_right_xoff} ${camera_right_yoff} ${camera_right_zoff} rpy=0 0 0 -> xyz=${camera_right_xoff} ${camera_right_yoff} ${camera_right_zoff} rpy=${camera_right_rotx} ${camera_right_roty} ${camera_right_rotz}; parent base_link -> camera_left_link
